File: keyboard_v1.0/cherry_mx_keys.kicad_sch (KiCad schematic)
At the start: 36 parts

Commit message: 2022.03.02. 18:05
Parts:
- removed D? (x18): DIODE, symbol Simulation_SPICE:DIODE
- added D? (x18): LL4148, Diode_SMD:D_MiniMELF, symbol Diode:LL4148
- added R? (x5): 10K, symbol Device:R
Connections:
- net at SW?.1, SW?.2, SW?.2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: now also D?.2 (A), R?.2 (x2)
- net at SW?.1: now also D?.2 (A) (x14)
- net at SW?.1, SW?.2, SW?.2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: now also D?.2 (A), R?.2 (x2)
- net at SW?.2, SW?.2, SW?.2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: now also R?.2
- new net: D?.1 (K), D?.1 (K), D?.1 (K), D?.1 (K), D?.1 (K) (x3)
- new net: D?.1 (K), D?.1 (K), D?.1 (K)
- new net 1. column: R?.1
- new net 2. column: R?.1
- new net 3. column: R?.1
- new net 4. column: R?.1
- new net 5. column: R?.1
