File: keyboard_v1.0/esp32.kicad_sch (KiCad schematic)
At the start: 5 parts

Commit message: 2022.03.02. 18:05
Parts:
- C?: value C -> 0.1 F
- R?: value R -> 10k
Changed lines of the file:
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@@
     (in_bom yes) (on_board yes) (fields_autoplaced)
     (property "Reference" "R?" (id 0) (at 60.96 49.53 90))
-    (property "Value" "R" (id 1) (at 60.96 52.07 90))
+    (property "Value" "10k" (id 1) (at 60.96 52.07 90))
     (property "Footprint" "" (id 2) (at 60.96 57.658 90)
       (effects (font (size 1.27 1.27)) hide)
@@
       (effects (font (size 1.27 1.27)) (justify left))
     )
-    (property "Value" "C" (id 1) (at 62.23 63.4999 0)
+    (property "Value" "0.1 F" (id 1) (at 62.23 63.4999 0)
       (effects (font (size 1.27 1.27)) (justify left))
     )
