File: keyboard_v1.0/keyboard_v1.0.kicad_pcb (KiCad board)
At the start: 2 copper layers, 8.2 x 5 mm, 25 parts, among them M3 MountingHole_3.2mm_M3

Commit message: 2022.03.02. 18:05
Parts:
- removed IC**: SOT230P700X180-4N, lm1117:SOT230P700X180-4N
- added REF**: lm1117 - sot223, lm1117:lm1117 - sot223, F.Cu at (105.8, 39.0)
