File: keyboard_v1.0/keyboard_v1.0.kicad_sch (KiCad schematic)
At the start: 0 parts

Commit message: 2022.02.23. 22:56
Other:
- added sheet Cherry MX keys (cherry_mx_keys.kicad_sch)
- added sheet ESP32 (esp32.kicad_sch)
- added sheet USB-C (usb-c.kicad_sch)
- added sheet WS2812B (ws2812b.kicad_sch)
