File: keyboard_v1.0/usb-c.kicad_sch (KiCad schematic)
At the start: 5 parts

Commit message: 2022.03.02. 18:05
Parts:
- added BT?: Battery_Cell, symbol Device:Battery_Cell
- added C? (x2): 4.7u, symbol Device:C
- added D?: LED, symbol Device:LED
- added F?: 1812L, symbol Device:Polyfuse
- added R?: 2K, symbol Device:R
- added R?: 5.1K, symbol Device:R
- added TP?: TestPoint, symbol Connector:TestPoint
- added U?: MCP73831-2-OT, Package_TO_SOT_SMD:SOT-23-5, symbol Battery_Management:MCP73831-2-OT
- C?: value C -> 100u
- C?: value C -> 10u
- R?: value R -> 5.1K
Connections:
- net +5V: now also C?.1, D?.2 (A), F?.2, U?.4 (VDD); no longer P?.A4 (VBUS), P?.A9 (VBUS), P?.B4 (VBUS), P?.B5 (VCONN), P?.B9 (VBUS)
- net GND: now also BT?.2 (-), C?.2, C?.2, R?.2, U?.2 (VSS)
- new net: R?.1, U?.5 (PROG)
- new net: R?.2, U?.1 (STAT)
- new net: BT?.1 (+), C?.1, U?.3 (VBAT)
- new net: F?.1, P?.A4 (VBUS), P?.A9 (VBUS), P?.B4 (VBUS), P?.B9 (VBUS)
- new net: P?.B5 (VCONN), TP?.1
- new net: D?.1 (K), R?.1
