File: keyboard_v1.0/ws2812b.kicad_sch (KiCad schematic)
At the start: 36 parts

Commit message: 2022.03.02. 18:05
Parts:
- C? (x18): value C -> 0.1u
Changed lines of the file:
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@@
       (effects (font (size 1.27 1.27)) (justify left))
     )
-    (property "Value" "C" (id 1) (at 168.91 137.1599 0)
+    (property "Value" "0.1u" (id 1) (at 168.91 137.1599 0)
       (effects (font (size 1.27 1.27)) (justify left))
     )
@@
       (effects (font (size 1.27 1.27)) (justify left))
     )
-    (property "Value" "C" (id 1) (at 69.85 83.8199 0)
+    (property "Value" "0.1u" (id 1) (at 69.85 83.8199 0)
       (effects (font (size 1.27 1.27)) (justify left))
     )
@@
       (effects (font (size 1.27 1.27)) (justify left))
     )
-    (property "Value" "C" (id 1) (at 107.95 83.8199 0)
+    (property "Value" "0.1u" (id 1) (at 107.95 83.8199 0)
       (effects (font (size 1.27 1.27)) (justify left))
     )
@@
       (effects (font (size 1.27 1.27)) (justify left))
     )
-    (property "Value" "C" (id 1) (at 54.61 24.1299 0)
+    (property "Value" "0.1u" (id 1) (at 54.61 24.1299 0)
       (effects (font (size 1.27 1.27)) (justify left))
     )
@@
       (effects (font (size 1.27 1.27)) (justify left))
     )
-    (property "Value" "C" (id 1) (at 92.71 24.1299 0)
+    (property "Value" "0.1u" (id 1) (at 92.71 24.1299 0)
       (effects (font (size 1.27 1.27)) (justify left))
     )
@@
       (effects (font (size 1.27 1.27)) (justify left))
     )
-    (property "Value" "C" (id 1) (at 54.61 99.0599 0)
+    (property "Value" "0.1u" (id 1) (at 54.61 99.0599 0)
       (effects (font (size 1.27 1.27)) (justify left))
     )
@@
       (effects (font (size 1.27 1.27)) (justify left))
     )
-    (property "Value" "C" (id 1) (at 168.91 24.1299 0)
+    (property "Value" "0.1u" (id 1) (at 168.91 24.1299 0)
       (effects (font (size 1.27 1.27)) (justify left))
     )
@@
       (effects (font (size 1.27 1.27)) (justify left))
     )
-    (property "Value" "C" (id 1) (at 207.01 137.1599 0)
+    (property "Value" "0.1u" (id 1) (at 207.01 137.1599 0)
       (effects (font (size 1.27 1.27)) (justify left))
     )
@@
       (effects (font (size 1.27 1.27)) (justify left))
     )
-    (property "Value" "C" (id 1) (at 168.91 99.0599 0)
+    (property "Value" "0.1u" (id 1) (at 168.91 99.0599 0)
       (effects (font (size 1.27 1.27)) (justify left))
     )
@@
       (effects (font (size 1.27 1.27)) (justify left))
     )
-    (property "Value" "C" (id 1) (at 92.71 99.0599 0)
+    (property "Value" "0.1u" (id 1) (at 92.71 99.0599 0)
       (effects (font (size 1.27 1.27)) (justify left))
     )
@@
       (effects (font (size 1.27 1.27)) (justify left))
     )
-    (property "Value" "C" (id 1) (at 207.01 99.0599 0)
+    (property "Value" "0.1u" (id 1) (at 207.01 99.0599 0)
       (effects (font (size 1.27 1.27)) (justify left))
     )
@@
       (effects (font (size 1.27 1.27)) (justify left))
     )
-    (property "Value" "C" (id 1) (at 130.81 99.0599 0)
+    (property "Value" "0.1u" (id 1) (at 130.81 99.0599 0)
       (effects (font (size 1.27 1.27)) (justify left))
     )
@@
       (effects (font (size 1.27 1.27)) (justify left))
     )
-    (property "Value" "C" (id 1) (at 130.81 137.1599 0)
+    (property "Value" "0.1u" (id 1) (at 130.81 137.1599 0)
       (effects (font (size 1.27 1.27)) (justify left))
     )
@@
       (effects (font (size 1.27 1.27)) (justify left))
     )
-    (property "Value" "C" (id 1) (at 222.25 83.8199 0)
+    (property "Value" "0.1u" (id 1) (at 222.25 83.8199 0)
       (effects (font (size 1.27 1.27)) (justify left))
     )
@@
       (effects (font (size 1.27 1.27)) (justify left))
     )
-    (property "Value" "C" (id 1) (at 146.05 83.8199 0)
+    (property "Value" "0.1u" (id 1) (at 146.05 83.8199 0)
       (effects (font (size 1.27 1.27)) (justify left))
     )
@@
       (effects (font (size 1.27 1.27)) (justify left))
     )
-    (property "Value" "C" (id 1) (at 207.01 24.1299 0)
+    (property "Value" "0.1u" (id 1) (at 207.01 24.1299 0)
       (effects (font (size 1.27 1.27)) (justify left))
     )
@@
       (effects (font (size 1.27 1.27)) (justify left))
     )
-    (property "Value" "C" (id 1) (at 184.15 83.8199 0)
+    (property "Value" "0.1u" (id 1) (at 184.15 83.8199 0)
       (effects (font (size 1.27 1.27)) (justify left))
     )
@@
       (effects (font (size 1.27 1.27)) (justify left))
     )
-    (property "Value" "C" (id 1) (at 130.81 24.1299 0)
-      (effects (font (size 1.27 1.27)) (justify left))
-    )
+    (property "Value" "0.1u" (id 1) (at 130.81 24.1299 0)
+      (effects (font (size 1.27 1.27)) (justify left))
+    )
